Commit message: stl import test

File: model/khrsugihara/khrsugihara.urdf (robot description, URDF)
Before this commit: robot khrsugihara, 24 links, 23 joints
Links:
- removed link LLEG_LINK3
- removed link LLEG_LINK4
- removed link RLEG_LINK2
- removed link RLEG_LINK3
- removed link RLEG_LINK4
- link LLEG_LINK2: geometry collision mesh filename=package://kxr_robot_description/model/khrsugihara/mesh/real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 scale=0.001 0.001 0.001; visual mesh filename=package://kxr_robot_description/model/khrsugihara/mesh/real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 scale=0.001 0.001 0.001
Joints:
- removed joint LLEG_JOINT3
- removed joint LLEG_JOINT4
- removed joint RLEG_JOINT2
- removed joint RLEG_JOINT3
- removed joint RLEG_JOINT4

Commit message: add passive wheels at heel in khrsugihara

File: model/khrsugihara/khrsugihara.urdf (robot description, URDF)
Before this commit: robot khrsugihara, 19 links, 18 joints
Links:
- removed link bodyset93922848311048
- added link BASE_LINK, mass 0.512289; collision mesh filename=package://kxr_robot_description/model/khrsugihara/mesh/simp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 scale=1 1 1; visual mesh filename=package://kxr_robot_description/model/khrsugihara/mesh/simp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 scale=1 1 1
- added link LLEG_LINK_WHEEL1, mass 0.059469; collision mesh filename=package://kxr_robot_description/model/khrsugihara/mesh/real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 scale=0.001 0.001 0.001; visual mesh filename=package://kxr_robot_description/model/khrsugihara/mesh/real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 scale=0.001 0.001 0.001
- added link LLEG_LINK_WHEEL2, mass 0.059469; collision mesh filename=package://kxr_robot_description/model/khrsugihara/mesh/real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 scale=0.001 0.001 0.001; visual mesh filename=package://kxr_robot_description/model/khrsugihara/mesh/real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 scale=0.001 0.001 0.001
- added link RLEG_LINK2, mass 0.059469; collision mesh filename=package://kxr_robot_description/model/khrsugihara/mesh/real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 scale=0.001 0.001 0.001; visual mesh filename=package://kxr_robot_description/model/khrsugihara/mesh/real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 scale=0.001 0.001 0.001
- added link RLEG_LINK_WHEEL1, mass 0.059469; collision mesh filename=package://kxr_robot_description/model/khrsugihara/mesh/real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 scale=0.001 0.001 0.001; visual mesh filename=package://kxr_robot_description/model/khrsugihara/mesh/real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 scale=0.001 0.001 0.001
- added link RLEG_LINK_WHEEL2, mass 0.059469; collision mesh filename=package://kxr_robot_description/model/khrsugihara/mesh/real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 scale=0.001 0.001 0.001; visual mesh filename=package://kxr_robot_description/model/khrsugihara/mesh/real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 scale=0.001 0.001 0.001
Joints:
- added joint LLEG_JOINT3: type continuous, parent LLEG_LINK2, child LLEG_LINK_WHEEL1, origin xyz=-0.092 0.051 -0.0125 rpy=0 -0 0 , axis 0 1 0, limit lower=-3.14159 upper=3.14159 effort=100 velocity=0.5
- added joint LLEG_JOINT4: type continuous, parent LLEG_LINK2, child LLEG_LINK_WHEEL2, origin xyz=-0.092 0.020 -0.0125 rpy=0 -0 0 , axis 0 1 0, limit lower=-3.14159 upper=3.14159 effort=100 velocity=0.5
- added joint RLEG_JOINT2: type continuous, parent RLEG_LINK1, child RLEG_LINK2, origin xyz=0 0 -0.065 rpy=0 -0 0 , axis 0 1 0, limit lower=-3.14159 upper=3.14159 effort=100 velocity=0.5
- added joint RLEG_JOINT3: type continuous, parent RLEG_LINK2, child RLEG_LINK_WHEEL1, origin xyz=-0.092 -0.020 -0.0125 rpy=0 -0 0 , axis 0 1 0, limit lower=-3.14159 upper=3.14159 effort=100 velocity=0.5
- added joint RLEG_JOINT4: type continuous, parent RLEG_LINK2, child RLEG_LINK_WHEEL2, origin xyz=-0.092 -0.051 -0.0125 rpy=0 -0 0 , axis 0 1 0, limit lower=-3.14159 upper=3.14159 effort=100 velocity=0.5
- joint HEAD_JOINT0: parent bodyset93922848311048 -> BASE_LINK
- joint LARM_JOINT0: parent bodyset93922848311048 -> BASE_LINK
- joint LLEG_JOINT0: parent bodyset93922848311048 -> BASE_LINK
- joint RARM_JOINT0: parent bodyset93922848311048 -> BASE_LINK
- joint RLEG_JOINT0: parent bodyset93922848311048 -> BASE_LINK

Commit message: modify mass of wheel

File: model/khrsugihara/khrsugihara.urdf (robot description, URDF)
Before this commit: robot khrsugihara, 24 links, 23 joints
Links:
- link LLEG_LINK_WHEEL1: mass 0.059469 -> 0.025
- link LLEG_LINK_WHEEL2: mass 0.059469 -> 0.025
- link RLEG_LINK_WHEEL1: mass 0.059469 -> 0.025
- link RLEG_LINK_WHEEL2: mass 0.059469 -> 0.025

Commit message: add birotor mesh to urdf

File: model/khrsugihara/khrsugihara.urdf (robot description, URDF)
Before this commit: robot khrsugihara, 24 links, 23 joints
Links:
- added link BIROTOR_UNIT, mass 1.4; collision mesh filename=package://kxr_robot_description/model/khrsugihara/mesh/real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 scale=0.001 0.001 0.001; visual mesh filename=package://kxr_robot_description/model/khrsugihara/mesh/real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 scale=0.001 0.001 0.001
- link LLEG_LINK2: mass 0.059469 -> 0.23
- link RLEG_LINK2: mass 0.059469 -> 0.23
Joints:
- added joint BIROTOR_UNIT_JOINT: type fixed, parent BASE_LINK, child BIROTOR_UNIT, origin xyz=0 0 0 rpy=0 -0 0 

Commit message: update positions and add docking hand, trirotor

File: model/khrsugihara/khrsugihara.urdf (robot description, URDF)
Before this commit: robot khrsugihara, 25 links, 24 joints
Joints:
- joint BIROTOR_UNIT_JOINT: origin xyz=0 0 0 rpy=0 -0 0  -> xyz=-0.0565 0 0.040 rpy=0 -0 0 

Commit message: add update khrsugihara to trirotor model

File: model/khrsugihara/khrsugihara.urdf (robot description, URDF)
Before this commit: robot khrsugihara, 25 links, 24 joints
Links:
- removed link BIROTOR_UNIT
- added link DOCKING_PIPE, mass 1.4; collision mesh filename=package://kxr_robot_description/model/khrsugihara/mesh/real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 scale=0.001 0.001 0.001; visual mesh filename=package://kxr_robot_description/model/khrsugihara/mesh/real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 scale=0.001 0.001 0.001
- added link TRIROTOR_UNIT, mass 1.4; collision mesh filename=package://kxr_robot_description/model/khrsugihara/mesh/real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 scale=0.001 0.001 0.001; visual mesh filename=package://kxr_robot_description/model/khrsugihara/mesh/real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 scale=0.001 0.001 0.001
Joints:
- removed joint BIROTOR_UNIT_JOINT
- added joint DOCKING_PIPE_JOINT: type continuous, parent BASE_LINK, child DOCKING_PIPE, origin xyz=-0.0565 0 0.040 rpy=0 -0 0 , limit lower=-3.14159 upper=3.14159 effort=100 velocity=0.5
- added joint TRIROTOR_UNIT_JOINT: type continuous, parent DOCKING_PIPE, child TRIROTOR_UNIT, origin xyz=-0.045 0 0.083 rpy=0 -0 0 , limit lower=-3.14159 upper=3.14159 effort=100 velocity=0.5

Commit message: update centroid of trirotor and docking pipe weight

File: model/khrsugihara/khrsugihara.urdf (robot description, URDF)
Before this commit: robot khrsugihara, 26 links, 25 joints
Links:
- link DOCKING_PIPE: mass 1.4 -> 0.2
- link TRIROTOR_UNIT: mass 1.4 -> 1.7
Joints:
- joint DOCKING_PIPE_JOINT: limit lower=-3.14159 upper=3.14159 effort=100 velocity=0.5 -> (none); type continuous -> fixed
- joint TRIROTOR_UNIT_JOINT: limit lower=-3.14159 upper=3.14159 effort=100 velocity=0.5 -> (none); type continuous -> fixed
