Commit message: update mass of docking pipe

File: model/khrsugihara/khrsugihara-tri-tilt.urdf (robot description, URDF)
Before this commit: robot khrsugihara, 26 links, 25 joints
Links:
- link DOCKING_PIPE: mass 0.2 -> 0.104

File: model/khrsugihara/khrsugihara.urdf (robot description, URDF)
Before this commit: robot khrsugihara, 26 links, 25 joints
Links:
- link DOCKING_PIPE: mass 0.2 -> 0.2122

Commit message: update trirotor param

File: model/khrsugihara/khrsugihara-tri-tilt.urdf (robot description, URDF)
Before this commit: robot khrsugihara, 26 links, 25 joints
Links:
- link TRIROTOR_UNIT: mass 1.7 -> 1.47

File: model/kxr_flight_unit_tri/kxr_flight_unit_tri.urdf (robot description, URDF)
Before this commit: robot kxr_flight_unit_tri, 1 links, 0 joints
Links:
- link BASE_LINK: mass 1.7 -> 1.47
