Commit message: rename birotor and trirotor to flight_unit to use in the same function

File: model/khrsugihara/khrsugihara-birotor.urdf (robot description, URDF)
Before this commit: robot khrsugihara, 25 links, 24 joints
Links:
- removed link BIROTOR_UNIT
- added link FLIGHT_UNIT, mass 1.4; collision mesh filename=package://kxr_robot_description/model/khrsugihara/mesh/real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 scale=0.001 0.001 0.001; visual mesh filename=package://kxr_robot_description/model/khrsugihara/mesh/real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 scale=0.001 0.001 0.001
Joints:
- removed joint BIROTOR_UNIT_JOINT
- added joint FLIGHT_UNIT_JOINT: type fixed, parent BASE_LINK, child FLIGHT_UNIT, origin xyz=-0.0565 0 0.040 rpy=0 -0 0 

File: model/khrsugihara/khrsugihara-tri-tilt.urdf (robot description, URDF)
Before this commit: robot khrsugihara, 26 links, 25 joints
Links:
- removed link TRIROTOR_UNIT
- added link FLIGHT_UNIT, mass 1.47; collision mesh filename=package://kxr_robot_description/model/khrsugihara/mesh/real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 scale=0.001 0.001 0.001; visual mesh filename=package://kxr_robot_description/model/khrsugihara/mesh/real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 scale=0.001 0.001 0.001
Joints:
- removed joint TRIROTOR_UNIT_JOINT
- added joint FLIGHT_UNIT_JOINT: type fixed, parent DOCKING_PIPE, child FLIGHT_UNIT, origin xyz=-0.06844 0 -0.00098 rpy=0 -0.314159 0 

File: model/khrsugihara/khrsugihara.urdf (robot description, URDF)
Before this commit: robot khrsugihara, 26 links, 25 joints
Links:
- removed link TRIROTOR_UNIT
- added link FLIGHT_UNIT, mass 1.7; collision mesh filename=package://kxr_robot_description/model/khrsugihara/mesh/real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 scale=0.001 0.001 0.001; visual mesh filename=package://kxr_robot_description/model/khrsugihara/mesh/real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 scale=0.001 0.001 0.001
Joints:
- removed joint TRIROTOR_UNIT_JOINT
- added joint FLIGHT_UNIT_JOINT: type fixed, parent DOCKING_PIPE, child FLIGHT_UNIT, origin xyz=-0.045 0 0.083 rpy=0 -0 0 

Commit message: update birotor mass

File: model/khrsugihara/khrsugihara-birotor.urdf (robot description, URDF)
Before this commit: robot khrsugihara, 25 links, 24 joints
Links:
- link FLIGHT_UNIT: mass 1.4 -> 1.1546

Commit message: [urdf] update mass by model based and replace head with stereo camera head

File: model/khrsugihara/khrsugihara-birotor.urdf (robot description, URDF)
Before this commit: robot khrsugihara, 25 links, 24 joints
Links:
- added link HEAD_LINK1, mass 0.014361; collision mesh filename=package://kxr_robot_description/model/khrsugihara/mesh/real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 scale=0.001 0.001 0.001; visual mesh filename=package://kxr_robot_description/model/khrsugihara/mesh/real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 scale=0.001 0.001 0.001
- link BASE_LINK: mass 0.512289 -> 0.3375
- link HEAD_LINK0: geometry collision mesh filename=package://kxr_robot_description/model/khrsugihara/mesh/real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 scale=0.001 0.001 0.001; visual mesh filename=package://kxr_robot_description/model/khrsugihara/mesh/real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 scale=0.001 0.001 0.001
Joints:
- added joint HEAD_JOINT1: type continuous, parent HEAD_LINK0, child HEAD_LINK1, origin xyz=-0.0105 0 0.033 rpy=0 -0 0 , axis 0 1 0, limit lower=-3.14159 upper=3.14159 effort=100 velocity=0.5

File: model/khrsugihara/khrsugihara-tri-tilt.urdf (robot description, URDF)
Before this commit: robot khrsugihara, 26 links, 25 joints
Links:
- added link HEAD_LINK1, mass 0.014361; collision mesh filename=package://kxr_robot_description/model/khrsugihara/mesh/real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 scale=0.001 0.001 0.001; visual mesh filename=package://kxr_robot_description/model/khrsugihara/mesh/real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 scale=0.001 0.001 0.001
- link HEAD_LINK0: geometry collision mesh filename=package://kxr_robot_description/model/khrsugihara/mesh/real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 scale=0.001 0.001 0.001; visual mesh filename=package://kxr_robot_description/model/khrsugihara/mesh/real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 scale=0.001 0.001 0.001
Joints:
- added joint HEAD_JOINT1: type continuous, parent HEAD_LINK0, child HEAD_LINK1, origin xyz=-0.0105 0 0.033 rpy=0 -0 0 , axis 0 1 0, limit lower=-3.14159 upper=3.14159 effort=100 velocity=0.5

File: model/khrsugihara/khrsugihara.urdf (robot description, URDF)
Before this commit: robot khrsugihara, 26 links, 25 joints
Links:
- added link HEAD_LINK1, mass 0.014361; collision mesh filename=package://kxr_robot_description/model/khrsugihara/mesh/real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 scale=0.001 0.001 0.001; visual mesh filename=package://kxr_robot_description/model/khrsugihara/mesh/real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 scale=0.001 0.001 0.001
- link BASE_LINK: mass 0.512289 -> 0.3375
- link HEAD_LINK0: geometry collision mesh filename=package://kxr_robot_description/model/khrsugihara/mesh/real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 scale=0.001 0.001 0.001; visual mesh filename=package://kxr_robot_description/model/khrsugihara/mesh/real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 scale=0.001 0.001 0.001
Joints:
- added joint HEAD_JOINT1: type continuous, parent HEAD_LINK0, child HEAD_LINK1, origin xyz=-0.0105 0 0.033 rpy=0 -0 0 , axis 0 1 0, limit lower=-3.14159 upper=3.14159 effort=100 velocity=0.5

Commit message: [khrsugihara] update arm end coords

File: model/khrsugihara/khrsugihara-birotor.urdf (robot description, URDF)
Before this commit: robot khrsugihara, 26 links, 25 joints
Links:
- added link LARM_DUMMY_LINK
- added link RARM_DUMMY_LINK
Joints:
- added joint LARM_DUMMY: type continuous, parent LARM_LINK3, child LARM_DUMMY_LINK, origin xyz=0 0.045 -0.12 rpy=1.5693386615608387 1.0707957464058213 1.5691353259370653, axis -1 1.09536e-16 5.47679e-17, limit lower=-3.14159 upper=3.14159 effort=100 velocity=0.5
- added joint RARM_DUMMY: type continuous, parent RARM_LINK3, child RARM_DUMMY_LINK, origin xyz=0 -0.045 -0.12 rpy=-1.5693386615608387 1.0707957464058213 -1.5691353259370653, axis -1 1.09536e-16 5.47679e-17, limit lower=-3.14159 upper=3.14159 effort=100 velocity=0.5

File: model/khrsugihara/khrsugihara-tri-free.urdf (robot description, URDF)
Before this commit: robot khrsugihara, 28 links, 27 joints
Links:
- added link LARM_DUMMY_LINK
- added link RARM_DUMMY_LINK
Joints:
- added joint LARM_DUMMY: type continuous, parent LARM_LINK3, child LARM_DUMMY_LINK, origin xyz=0 0.045 -0.12 rpy=1.5693386615608387 1.0707957464058213 1.5691353259370653, axis -1 1.09536e-16 5.47679e-17, limit lower=-3.14159 upper=3.14159 effort=100 velocity=0.5
- added joint RARM_DUMMY: type continuous, parent RARM_LINK3, child RARM_DUMMY_LINK, origin xyz=0 -0.045 -0.12 rpy=-1.5693386615608387 1.0707957464058213 -1.5691353259370653, axis -1 1.09536e-16 5.47679e-17, limit lower=-3.14159 upper=3.14159 effort=100 velocity=0.5

File: model/khrsugihara/khrsugihara-tri-tilt.urdf (robot description, URDF)
Before this commit: robot khrsugihara, 27 links, 26 joints
Links:
- added link LARM_DUMMY_LINK
- added link RARM_DUMMY_LINK
Joints:
- added joint LARM_DUMMY: type continuous, parent LARM_LINK3, child LARM_DUMMY_LINK, origin xyz=0 0.045 -0.12 rpy=1.5693386615608387 1.0707957464058213 1.5691353259370653, axis -1 1.09536e-16 5.47679e-17, limit lower=-3.14159 upper=3.14159 effort=100 velocity=0.5
- added joint RARM_DUMMY: type continuous, parent RARM_LINK3, child RARM_DUMMY_LINK, origin xyz=0 -0.045 -0.12 rpy=-1.5693386615608387 1.0707957464058213 -1.5691353259370653, axis -1 1.09536e-16 5.47679e-17, limit lower=-3.14159 upper=3.14159 effort=100 velocity=0.5

File: model/khrsugihara/khrsugihara.urdf (robot description, URDF)
Before this commit: robot khrsugihara, 27 links, 26 joints
Links:
- added link LARM_DUMMY_LINK
- added link RARM_DUMMY_LINK
Joints:
- added joint LARM_DUMMY: type continuous, parent LARM_LINK3, child LARM_DUMMY_LINK, origin xyz=0 0.045 -0.12 rpy=1.5693386615608387 1.0707957464058213 1.5691353259370653, axis -1 1.09536e-16 5.47679e-17, limit lower=-3.14159 upper=3.14159 effort=100 velocity=0.5
- added joint RARM_DUMMY: type continuous, parent RARM_LINK3, child RARM_DUMMY_LINK, origin xyz=0 -0.045 -0.12 rpy=-1.5693386615608387 1.0707957464058213 -1.5691353259370653, axis -1 1.09536e-16 5.47679e-17, limit lower=-3.14159 upper=3.14159 effort=100 velocity=0.5
