Commit message: update khr model

File: model/khrsugihara/khrsugihara_yaw_lock_joint.urdf (robot description, URDF)
Before this commit: robot khrsugihara, 32 links, 31 joints
Links:
- added link flight_unit_dummy
- added link thrust_link1; collision mesh filename=package://kxr_robot_description/model/khrsugihara/mesh/real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 scale=0.001 0.001 0.001; visual mesh filename=package://kxr_robot_description/model/khrsugihara/mesh/real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 scale=0.001 0.001 0.001
- added link thrust_link2; collision mesh filename=package://kxr_robot_description/model/khrsugihara/mesh/real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 scale=0.001 0.001 0.001; visual mesh filename=package://kxr_robot_description/model/khrsugihara/mesh/real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 scale=0.001 0.001 0.001
- added link thrust_link3; collision mesh filename=package://kxr_robot_description/model/khrsugihara/mesh/real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 scale=0.001 0.001 0.001; visual mesh filename=package://kxr_robot_description/model/khrsugihara/mesh/real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 scale=0.001 0.001 0.001
- link FLIGHT_UNIT: mass 1.47 -> 1.1
- link LARM_DUMMY_LINK: mass None -> 0.001
- link LLEG_DUMMY_LINK_0: mass None -> 0.001
- link RARM_DUMMY_LINK: mass None -> 0.001
- link RLEG_DUMMY_LINK_0: mass None -> 0.001
Joints:
- added joint FLIGHT_UNIT_DUMMY_JOINT: type fixed, parent DOCKING_HAND, child flight_unit_dummy, origin xyz=0.08 0 0.096 rpy=0 -0 0 , axis 0 1 0
- added joint gimbal1: type continuous, parent FLIGHT_UNIT, child thrust_link1, origin xyz=0 0.2375 0.051 rpy=0 0 1.57, axis 1 0 0
- added joint gimbal2: type continuous, parent FLIGHT_UNIT, child thrust_link2, origin xyz=0 -0.2375 0.051 rpy=0 0 -1.57, axis 1 0 0
- added joint gimbal3: type continuous, parent FLIGHT_UNIT, child thrust_link3, origin xyz=-0.2975 0 0.051 rpy=0 0 3.14, axis 1 0 0
- joint FLIGHT_UNIT_JOINT: axis 0 1 0 -> (none); origin xyz=0 0 0.096 rpy=0 -0 0  -> (none); parent DOCKING_HAND -> flight_unit_dummy
