Commit message: add kxr_flight_unit_tri directory

File: model/kxr_flight_unit_tri/kxr_flight_unit_tri.urdf (robot description, URDF)
Before this commit: robot kxr_flight_unit_tri, 1 links, 0 joints
Links:
- link BASE_LINK: geometry collision mesh filename=package://kxr_robot_description/model/kxr_flight_unit_tri/m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 scale=0.001 0.001 0.001; visual mesh filename=package://kxr_robot_description/model/kxr_flight_unit_tri/m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 scale=0.001 0.001 0.001
